File: Capstone_Signal_Processing_PCB/Capstone_Signal_Processing.kicad_pcb (KiCad board)
At the start: 4 copper layers, 35.5 x 36.9 mm, 21 parts, among them J1 Conn_01x01, J2 Conn_01x01, J3 Conn_01x01, J4 Conn_01x04, J5 Conn_01x02, U1 AD4170-4BCPZ

Commit message: Fixes to Signal Processing PCB, Tx-Rx Added
Parts:
- added J6: Conn_01x02, Connector_JST:JST_XH_B2B-XH-AM_1x02_P2.50mm_Vertical, F.Cu at (131.6, 107.3)
- R1: value 10k -> 1M
- R2: value 20k -> 1M
- moved R1 7.13 mm to (138.1, 111.1), turned to -90 degrees
- moved R2 1.00 mm to (140.0, 104.2), turned to 180 degrees
- renumbered J1 to J1_CHX, J2 to J2_CHY, J3 to J3_CHZ
Connections:
- R1 pad 1: +5V -> +3.3V
- R1 pad 2: +3.3V -> /CS
- R2 pad 1: +3.3V -> Net-(U1-*SYNC_IN)
- R2 pad 2: GND -> +3.3V
- U1 pad 11: unconnected-(U1-*SYNC_IN-Pad11) -> Net-(U1-*SYNC_IN)
Routing:
- net /CS: track 9.60 -> 20.4 mm
- net +5V: track 26.2 -> 15.5 mm
- net +3.3V: track 26.9 -> 37.5 mm
- net GND: track 72.2 -> 80.6 mm
- net Net-(U1-*SYNC_IN): track 0.00 -> 6.42 mm
Other:
- board text added: "3V3-GND"
- board text added: "GND-5V"
- board text added: "SDI-SDO-CS-SCLK"

Commit message: Final Changes to ADC PCB
Parts:
- removed J1_CHX, J2_CHY, J3_CHZ: Conn_01x01, Connector_JST:JST_XH_B1B-XH-AM_1x01_P2.50mm_Vertical
- added J1: Conn_01x02, Connector_JST:JST_XH_B2B-XH-AM_1x02_P2.50mm_Vertical, F.Cu at (140.9, 85.1)
- added J2: Conn_01x02, Connector_JST:JST_XH_B2B-XH-AM_1x02_P2.50mm_Vertical, F.Cu at (149.8, 85.1)
- added J3: Conn_01x02, Connector_JST:JST_XH_B2B-XH-AM_1x02_P2.50mm_Vertical, F.Cu at (159.6, 89.3)
- added J7: Conn_01x02, Connector_JST:JST_XH_B2B-XH-AM_1x02_P2.50mm_Vertical, F.Cu at (134.1, 89.9)
- moved C4 0.30 mm to (141.4, 95.8)
Connections:
- U1 pad 2: unconnected-(U1-REFIN+-Pad2) -> /Ref+
- U1 pad 28: GND -> /CH_Z_GND
- U1 pad 3: unconnected-(U1-REFIN--Pad3) -> /Ref-(GND)
- U1 pad 30: GND -> /CH_Y_GND
- U1 pad 32: GND -> /CH_X_GND
Routing:
- net /Ref-(GND): track 0.00 -> 18.5 mm
- net /Ref+: track 0.00 -> 15.7 mm
- net /CH_Z_GND: track 0.00 -> 13.7 mm
- net /CH_Y_GND: track 0.00 -> 13.2 mm
- net /CH_X_GND: track 0.00 -> 12.2 mm
- net GND: track 80.6 -> 73.1 mm, vias 12 -> 9
- net /CH_X: track 16.3 -> 13.7 mm
- net /CH_Z: track 14.2 -> 15.6 mm
Other:
- board text added: "Ref+ Ref-"
- board text added: "X_GND X_SIG"
- board text added: "Y_GND Y_SIG"
- board text added: "Z_SIG Z_GND"
